File: DIY_Keyboard_PCB.sch (KiCad schematic (older format))
At the start: 27 parts, among them SW1 SW_Push, U1 ATmega32U4-AU, Y1 Crystal_GND24_Small

Commit message: Saved changes
Parts:
- FID1, FID2, FID3: footprint (none) -> Fiducial:Fiducial_0.5mm_Mask1mm
Changed lines of the file:
@@
 F 0 "FID1" H 2685 6046 50  0000 L CNN
 F 1 "Fiducial" H 2685 5955 50  0000 L CNN
-F 2 "" H 2600 6000 50  0001 C CNN
+F 2 "Fiducial:Fiducial_0.5mm_Mask1mm" H 2600 6000 50  0001 C CNN
 F 3 "~" H 2600 6000 50  0001 C CNN
 	1    2600 6000
@@
 F 0 "FID2" H 3435 6046 50  0000 L CNN
 F 1 "Fiducial" H 3435 5955 50  0000 L CNN
-F 2 "" H 3350 6000 50  0001 C CNN
+F 2 "Fiducial:Fiducial_0.5mm_Mask1mm" H 3350 6000 50  0001 C CNN
 F 3 "~" H 3350 6000 50  0001 C CNN
 	1    3350 6000
@@
 F 0 "FID3" H 4085 6046 50  0000 L CNN
 F 1 "Fiducial" H 4085 5955 50  0000 L CNN
-F 2 "" H 4000 6000 50  0001 C CNN
+F 2 "Fiducial:Fiducial_0.5mm_Mask1mm" H 4000 6000 50  0001 C CNN
 F 3 "~" H 4000 6000 50  0001 C CNN
 	1    4000 6000
