File: DIY_Keyboard_PCB.kicad_pcb (KiCad board)
At the start: 2 copper layers, 71.4 x 38.1 mm, 24 parts, among them SW1 SW_Push, U1 ATmega32U4-AU, Y1 Crystal_GND24_Small

Commit message: Finished - gerbers generated
Parts:
- added G***: LOGO, random-keyboard-parts:artwork, F.Cu at (125.4, 165.1)
Routing:
- net Net-(USB1-Pad6): track 0.00 -> 16.3 mm
- added copper zone on B.Cu, net GND
